File: pcb/tenkeyless-nofunctions.kicad_pcb (KiCad board)
At the start: 2 copper layers, 352.4 x 95.2 mm, 142 parts, among them SW1 TILDE, SW10 NUM_9, SW11 NUM_0, SW12 UNDRSCR, SW13 EQUAL, SW14 BCKSPC, SW15 INSRT, SW16 HOME, SW17 PG_UP, SW18 LTAB, SW19 KEY_Q, SW2 NUM_1, SW20 KEY_W, SW21 KEY_E, SW22 KEY_R, SW23 KEY_T, SW24 KEY_Y, SW25 KEY_U, SW26 KEY_I, SW27 KEY_O, SW28 KEY_P, SW29 OP_BRKT, SW3 NUM_2, SW30 CL_BRKT, SW31 BKSLSH, SW32 DELETE, SW33 END, SW34 PG_DN, SW35 CAPS, SW36 KEY_A, SW37 KEY_S, SW38 KEY_D, SW39 KEY_F, SW4 NUM_3, SW40 KEY_G, SW41 KEY_H, SW42 KEY_J, SW43 KEY_K, SW44 KEY_L, SW45 SEMICOLON, SW46 QUOTE, SW47 ENTER, SW48 LSHIFT, SW49 KEY_Z, SW5 NUM_4, SW50 KEY_X, SW51 KEY_C, SW52 KEY_V, SW53 KEY_B, SW54 KEY_N, SW55 KEY_M, SW56 COMMA, SW57 PERIOD, SW58 FWDSLSH, SW59 RSHIFT, SW6 NUM_5, SW60 UP, SW61 LCTRL, SW62 WIN, SW63 LALT, SW64 SPACE, SW65 RALT, SW66 RCTRL, SW67 FN, SW68 ESC, SW69 LEFT, SW7 NUM_6, SW70 DN, SW71 RIGHT, SW8 NUM_7, SW9 NUM_8

Commit message: flipped keymodule pins; now gotta figure out routing with as few jumps as possible
Parts:
- moved D48 2.48 mm to (40.4, 91.4)
- moved D61 2.47 mm to (30.7, 110.7)
- moved D35 2.42 mm to (35.6, 72.4)
- moved D64 2.38 mm to (150.0, 109.5)
- moved SW59 2.38 mm to (278.6, 85.7)
- moved SW64 2.38 mm to (150.0, 104.8)
- moved SW67 2.38 mm to (269.1, 104.8)
- moved SW35 2.38 mm to (35.7, 66.7)
- moved SW48 2.38 mm to (40.5, 85.7)
- moved SW61 2.38 mm to (31.0, 104.8)
- moved D62 2.38 mm to (54.8, 109.5)
- moved D63 2.38 mm to (78.6, 109.5)
- moved SW62 2.38 mm to (54.8, 104.8)
- moved SW63 2.38 mm to (78.6, 104.8)
- moved SW65 2.38 mm to (221.5, 104.8)
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Routing:
- net /COL0: track 25.8 -> 93.8 mm
- net Net-(D61-Pad1): track 0.00 -> 9.26 mm
- net Net-(D35-Pad1): track 0.00 -> 9.03 mm
- net Net-(D48-Pad1): track 0.00 -> 8.85 mm
- net Net-(D18-Pad1): track 11.2 -> 8.09 mm
