File: tenkeyless-nofunctions/tenkeyless-nofunctions.kicad_pcb (KiCad board)
At the start: 2 copper layers, 352.4 x 95.2 mm, 142 parts, among them SW1 TILDE, SW10 NUM_9, SW11 NUM_0, SW12 UNDRSCR, SW13 EQUAL, SW14 BCKSPC, SW15 INSRT, SW16 HOME, SW17 PG_UP, SW18 LTAB, SW19 KEY_Q, SW2 NUM_1, SW20 KEY_W, SW21 KEY_E, SW22 KEY_R, SW23 KEY_T, SW24 KEY_Y, SW25 KEY_U, SW26 KEY_I, SW27 KEY_O, SW28 KEY_P, SW29 OP_BRKT, SW3 NUM_2, SW30 CL_BRKT, SW31 BKSLSH, SW32 DELETE, SW33 END, SW34 PG_DN, SW35 CAPS, SW36 KEY_A, SW37 KEY_S, SW38 KEY_D, SW39 KEY_F, SW4 NUM_3, SW40 KEY_G, SW41 KEY_H, SW42 KEY_J, SW43 KEY_K, SW44 KEY_L, SW45 SEMICOLON, SW46 QUOTE, SW47 ENTER, SW48 LSHIFT, SW49 KEY_Z, SW5 NUM_4, SW50 KEY_X, SW51 KEY_C, SW52 KEY_V, SW53 KEY_B, SW54 KEY_N, SW55 KEY_M, SW56 COMMA, SW57 PERIOD, SW58 FWDSLSH, SW59 RSHIFT, SW6 NUM_5, SW60 UP, SW61 LCTRL, SW62 WIN, SW63 LALT, SW64 SPACE, SW65 RALT, SW66 RCTRL, SW67 FN, SW68 ESC, SW69 LEFT, SW7 NUM_6, SW70 DN, SW71 RIGHT, SW8 NUM_7, SW9 NUM_8

Commit message: did some organizing of the files before this got any more out of hand
Parts:
- moved D1 11.3 mm to (38.1, 27.3), turned to 270 degrees
- moved D2 11.3 mm to (57.1, 27.3), turned to 270 degrees
- moved D19 10.6 mm to (66.7, 47.8), turned to 270 degrees
Routing:
- net /COL0: track 93.8 -> 2.30 mm
- net /ROW4: track 19.1 -> 0.89 mm
- net Net-(D61-Pad1): track 9.26 -> 0.00 mm
- net Net-(D35-Pad1): track 9.03 -> 0.00 mm
- net Net-(D48-Pad1): track 8.85 -> 0.00 mm
- net Net-(D18-Pad1): track 8.09 -> 0.00 mm
- net Net-(D1-Pad1): track 8.04 -> 0.00 mm
- net /ROW2: track 0.00 -> 1.21 mm
- net /ROW0: track 0.00 -> 1.12 mm
- net /ROW1: track 0.00 -> 0.94 mm

Commit message: new tenkey board
Parts:
- SW1, SW10, SW11, SW12, SW13, SW14, SW15, SW16, SW17, SW18, SW19, SW2, SW20, SW21, SW22, SW23, SW24, SW25, SW26, SW27, SW28, SW29, SW3, SW30, SW31, SW32, SW33, SW34, SW35, SW36, SW37, SW38, SW39, SW4, SW40, SW41, SW42, SW43, SW44, SW45, SW46, SW47, SW48, SW49, SW5, SW50, SW51, SW52, SW53, SW54, SW55, SW56, SW57, SW58, SW59, SW6, SW60, SW61, SW62, SW63, SW64, SW65, SW66, SW67, SW68, SW69, SW7, SW70, SW71, SW8, SW9: footprint Custom:KEYMODULE_MX_PINS -> Keyboard:KEYMODULE_MX_PINS
- moved D1 12.6 mm to (28.7, 35.7), turned to 0 degrees
- moved D2 12.6 mm to (47.8, 35.7), turned to 0 degrees
Routing:
- net Net-(D35-Pad1): track 0.00 -> 1.21 mm
- net /ROW2: track 1.21 -> 0.00 mm
- net Net-(D61-Pad1): track 0.00 -> 1.12 mm
- net /ROW0: track 1.12 -> 0.00 mm
- net Net-(D48-Pad1): track 0.00 -> 0.94 mm
- net /ROW1: track 0.94 -> 0.00 mm
- net Net-(D1-Pad1): track 0.00 -> 0.89 mm
- net /ROW4: track 0.89 -> 0.00 mm
Other:
- net class Default: trace_width 0.254 -> 0.35
